Commit message: Mastering URDS, Xacro, bridge with Rviz2 and Gazebo

File: src/rosbot_description/urdf/materials.xacro (robot description, xacro)
@@ -1,6 +1,47 @@
-<?xml version="1.0" ?>
-<robot name="rosbot" xmlns:xacro="http://www.ros.org/wiki/xacro" >
-<material name="silver">
-  <color rgba="0.700 0.700 0.700 1.000"/>
-</material>
+<?xml version="1.0"?>
+<!--
+  XML declaration
+  指定 XML 版本。URDF / Xacro 文件本质都是 XML。
+-->
+<robot name="rosbot" xmlns:xacro="http://www.ros.org/wiki/xacro">
+  <!--
+  robot:
+    URDF/Xacro 文件的根节点。
+  name="rosbot":
+    机器人模型名称。在 ROS / Gazebo / RViz 中会作为模型标识。
+  xmlns:xacro="http://www.ros.org/wiki/xacro":
+    声明 xacro 的 XML namespace（命名空间）。
+    作用：
+    允许在该文件中使用 xacro 的扩展语法，例如：
+        <xacro:property>
+        <xacro:macro>
+        <xacro:include>
+        <xacro:if>
+    本文件虽然暂时没有使用 xacro 指令，
+    但几乎所有 ROS2 机器人描述文件都会默认声明该 namespace，
+    方便后续扩展。
+-->
+  <material name="silver">
+    <!--
+    material:
+      定义一个可复用的材质。
+    name="silver":
+      材质名称。
+      在 link 的 visual 中可以通过：
+          <material name="silver"/>
+      来复用该材质。
+  -->
+    <color rgba="0.700 0.700 0.700 1.000" />
+    <!--
+      color:
+        定义材质颜色。
+      rgba:
+        Red   Green   Blue   Alpha
+      取值范围：
+        0.0 ~ 1.0
+      本例：
+        0.700 0.700 0.700  → 银灰色
+        1.000              → 完全不透明
+    -->
+  </material>
 </robot>

File: src/rosbot_description/urdf/rosbot.xacro (robot description, xacro)
@@ -1,109 +1,119 @@
-<?xml version="1.0" ?>
+<?xml version="1.0"?>
+<!-- XML声明 -->
 <robot name="rosbot" xmlns:xacro="http://www.ros.org/wiki/xacro">
-<xacro:include filename="$(find rosbot_description)/urdf/materials.xacro" />
-<xacro:include filename="$(find rosbot_description)/urdf/rosbot.ros2control" />
-<xacro:include filename="$(find rosbot_description)/urdf/rosbot.gazebo" />
-<link name="base_footprint"/>
-<link name="base_link">
-  <inertial>
-    <origin xyz="0.004279734419382094 0.0 0.05375741183973183" rpy="0 0 0"/>
-    <mass value="2.34056579648116"/>
-    <inertia ixx="0.008048" iyy="0.008642" izz="0.014848" ixy="-0.0" iyz="0.0" ixz="-0.000438"/>
-  </inertial>
-  <visual>
-    <origin xyz="0 0 0" rpy="0 0 0"/>
-    <geometry>
-      <mesh filename="file://$(find rosbot_description)/meshes/base_link.stl" scale="0.001 0.001 0.001"/>
-    </geometry>
-    <material name="silver"/>
-  </visual>
-  <collision>
-    <origin xyz="0 0 0" rpy="0 0 0"/>
-    <geometry>
-      <mesh filename="file://$(find rosbot_description)/meshes/base_link.stl" scale="0.001 0.001 0.001"/>
-    </geometry>
-  </collision>
-</link>
-<link name="right_wheel_1">
-  <inertial>
-    <origin xyz="-5.790023100122029e-18 -0.012499999999999997 3.7252903539730653e-10" rpy="0 0 0"/>
-    <mass value="0.1826050729899067"/>
-    <inertia ixx="0.000124" iyy="0.000228" izz="0.000124" ixy="-0.0" iyz="-0.0" ixz="0.0"/>
-  </inertial>
-  <visual>
-    <origin xyz="-0.0 0.1 -0.05" rpy="0 0 0"/>
-    <geometry>
-      <mesh filename="file://$(find rosbot_description)/meshes/right_wheel_1.stl" scale="0.001 0.001 0.001"/>
-    </geometry>
-    <material name="silver"/>
-  </visual>
-  <collision>
-    <origin xyz="-0.0 0.1 -0.05" rpy="0 0 0"/>
-    <geometry>
-      <mesh filename="file://$(find rosbot_description)/meshes/right_wheel_1.stl" scale="0.001 0.001 0.001"/>
-    </geometry>
-  </collision>
-</link>
-<link name="left_wheel_1">
-  <inertial>
-    <origin xyz="1.737006930036608e-17 0.012499999999999997 3.725290284584126e-10" rpy="0 0 0"/>
-    <mass value="0.18260507298990675"/>
-    <inertia ixx="0.000124" iyy="0.000228" izz="0.000124" ixy="-0.0" iyz="0.0" ixz="0.0"/>
-  </inertial>
-  <visual>
-    <origin xyz="-0.0 -0.1 -0.05" rpy="0 0 0"/>
-    <geometry>
-      <mesh filename="file://$(find rosbot_description)/meshes/left_wheel_1.stl" scale="0.001 0.001 0.001"/>
-    </geometry>
-    <material name="silver"/>
-  </visual>
-  <collision>
-    <origin xyz="-0.0 -0.1 -0.05" rpy="0 0 0"/>
-    <geometry>
-      <mesh filename="file://$(find rosbot_description)/meshes/left_wheel_1.stl" scale="0.001 0.001 0.001"/>
-    </geometry>
-  </collision>
-</link>
-<link name="lidar_1">
-  <inertial>
-    <origin xyz="0.0 0.0 0.010000000000000009" rpy="0 0 0"/>
-    <mass value="0.0754575997873079"/>
-    <inertia ixx="1.9e-05" iyy="1.9e-05" izz="3.3e-05" ixy="0.0" iyz="0.0" ixz="0.0"/>
-  </inertial>
-  <visual>
-    <origin xyz="-0.05 -0.0 -0.21" rpy="0 0 0"/>
-    <geometry>
-      <mesh filename="file://$(find rosbot_description)/meshes/lidar_1.stl" scale="0.001 0.001 0.001"/>
-    </geometry>
-    <material name="silver"/>
-  </visual>
-  <collision>
-    <origin xyz="-0.05 -0.0 -0.21" rpy="0 0 0"/>
-    <geometry>
-      <mesh filename="file://$(find rosbot_description)/meshes/lidar_1.stl" scale="0.001 0.001 0.001"/>
-    </geometry>
-  </collision>
-</link>
-<joint name="base_joint" type="fixed">
-  <origin xyz="0.0 0.0 0.0" rpy="0 0 0"/>
-  <parent link="base_footprint"/>
-  <child link="base_link"/>
-</joint>
-<joint name="right_wheel_joint" type="continuous">
-  <origin xyz="0.0 -0.1 0.05" rpy="0 0 0"/>
-  <parent link="base_link"/>
-  <child link="right_wheel_1"/>
-  <axis xyz="0.0 1.0 0.0"/>
-</joint>
-<joint name="left_wheel_joint" type="continuous">
-  <origin xyz="0.0 0.1 0.05" rpy="0 0 0"/>
-  <parent link="base_link"/>
-  <child link="left_wheel_1"/>
-  <axis xyz="0.0 1.0 0.0"/>
-</joint>
-<joint name="lidar_joint" type="fixed">
-  <origin xyz="0.05 0.0 0.21" rpy="0 0 0"/>
-  <parent link="base_link"/>
-  <child link="lidar_1"/>
-</joint>
+  <!--
+robot: URDF / Xacro 根节点
+name: 机器人模型名称
+xmlns:xacro: 声明 xacro 命名空间，允许使用 <xacro:*> 指令
+-->
+  <!-- 引入其他xacro文件（模块化设计） -->
+  <xacro:include filename="$(find rosbot_description)/urdf/materials.xacro" />
+  <!-- 材质定义 -->
+  <xacro:include filename="$(find rosbot_description)/urdf/rosbot.ros2control" />
+  <!-- ros2_control 插件配置（电机控制接口） -->
+  <xacro:include filename="$(find rosbot_description)/urdf/rosbot.gazebo" />
+  <!-- Gazebo 仿真插件配置 -->
+  <link name="base_footprint" />
+  <!--
+base_footprint:
+机器人在地面的参考坐标系
+通常：
+z = 0
+用于 navigation / TF tree
+-->
+  <link name="base_link">
+    <!--
+base_link:
+机器人主体坐标系
+机器人动力学 / 传感器 / 控制的核心frame
+-->
+    <inertial>
+      <!--
+  惯性参数（动力学仿真用）
+  Gazebo / physics engine 必须
+  -->
+      <origin xyz="0.004279734419382094 0.0 0.05375741183973183" rpy="0 0 0" />
+      <!-- 质心位置 -->
+      <mass value="2.34056579648116" />
+      <!-- 质量 kg -->
+      <inertia ixx="0.008048" iyy="0.008642" izz="0.014848"
+        ixy="-0.0" iyz="0.0" ixz="-0.000438" />
+      <!-- 惯性矩阵 -->
+    </inertial>
+    <visual>
+      <!-- RViz / Gazebo 显示模型 -->
+      <origin xyz="0 0 0" rpy="0 0 0" />
+      <geometry>
+        <mesh filename="file://$(find rosbot_description)/meshes/base_link.stl"
+          scale="0.001 0.001 0.001" />
+        <!--
+      mesh: 3D模型
+      scale: STL通常mm，需要缩放到m
+      -->
+      </geometry>
+      <material name="silver" />
+      <!-- 使用 materials.xacro 中定义的材质 -->
+    </visual>
+    <collision>
+      <!-- 物理碰撞模型 -->
+      <origin xyz="0 0 0" rpy="0 0 0" />
+      <geometry>
+        <mesh filename="file://$(find rosbot_description)/meshes/base_link.stl"
+          scale="0.001 0.001 0.001" />
+      </geometry>
+    </collision>
+  </link>
+  <link name="right_wheel_1">
+    <!-- 右轮 link -->
+    <inertial> ... </inertial>
+    <visual>
+      <!-- 轮子的可视模型 -->
+    </visual>
+    <collision>
+      <!-- 轮子的碰撞模型 -->
+    </collision>
+  </link>
+  <link name="left_wheel_1">
+    <!-- 左轮 link -->
+  </link>
+  <link name="lidar_1">
+    <!-- LiDAR 传感器模型 -->
+  </link>
+  <joint name="base_joint" type="fixed">
+    <!--
+joint: 连接两个link
+type="fixed"
+表示两个link刚性连接
+-->
+    <origin xyz="0.0 0.0 0.0" rpy="0 0 0" />
+    <parent link="base_footprint" />
+    <!-- 父坐标系 -->
+    <child link="base_link" />
+    <!-- 子坐标系 -->
+  </joint>
+  <joint name="right_wheel_joint" type="continuous">
+    <!--
+continuous:
+无限旋转关节
+适用于轮子
+-->
+    <origin xyz="0.0 -0.1 0.05" rpy="0 0 0" />
+    <!-- 轮子相对于base_link的位置 -->
+    <parent link="base_link" />
+    <child link="right_wheel_1" />
+    <axis xyz="0.0 1.0 0.0" />
+    <!-- 轮子旋转轴 -->
+  </joint>
+  <joint name="left_wheel_joint" type="continuous">
+    <origin xyz="0.0 0.1 0.05" rpy="0 0 0" />
+    <parent link="base_link" />
+    <child link="left_wheel_1" />
+    <axis xyz="0.0 1.0 0.0" />
+  </joint>
+  <joint name="lidar_joint" type="fixed">
+    <!-- LiDAR 固定安装 -->
+    <origin xyz="0.05 0.0 0.21" rpy="0 0 0" />
+    <parent link="base_link" />
+    <child link="lidar_1" />
+  </joint>
 </robot>

File: src/rrbot_description/urdf/rrbot.materials.xacro (robot description, xacro)
@@ -6,29 +6,29 @@
 <robot>
   <material name="black">
-    <color rgba="0.0 0.0 0.0 1.0"/>
+    <color rgba="0.0 0.0 0.0 1.0" />
   </material>
   <material name="blue">
-    <color rgba="0.0 0.0 0.8 1.0"/>
+    <color rgba="0.0 0.0 0.8 1.0" />
   </material>
   <material name="green">
-    <color rgba="0.0 0.8 0.0 1.0"/>
+    <color rgba="0.0 0.8 0.0 1.0" />
   </material>
   <material name="grey">
-    <color rgba="0.2 0.2 0.2 1.0"/>
+    <color rgba="0.2 0.2 0.2 1.0" />
   </material>
   <material name="orange">
-    <color rgba="${255/255} ${108/255} ${10/255} 1.0"/>
+    <color rgba="${255/255} ${108/255} ${10/255} 1.0" />
   </material>
   <material name="brown">
-    <color rgba="${222/255} ${207/255} ${195/255} 1.0"/>
+    <color rgba="${222/255} ${207/255} ${195/255} 1.0" />
   </material>
   <material name="red">
-    <color rgba="0.8 0.0 0.0 1.0"/>
+    <color rgba="0.8 0.0 0.0 1.0" />
   </material>
   <material name="yellow">
-    <color rgba="1.0 1.0 0.0 1.0"/>
+    <color rgba="1.0 1.0 0.0 1.0" />
   </material>
   <material name="white">
-    <color rgba="1.0 1.0 1.0 1.0"/>
+    <color rgba="1.0 1.0 1.0 1.0" />
   </material>
 </robot>

File: src/rrbot_description/urdf/rrbot_description.urdf.xacro (robot description, xacro)
@@ -2,112 +2,119 @@
 <robot xmlns:xacro="http://www.ros.org/wiki/xacro">
   <xacro:macro name="rrbot" params="parent prefix *origin">
-  <!-- Constants for robot dimensions -->
-  <xacro:property name="mass" value="1" /> <!-- arbitrary value for mass -->
-  <xacro:property name="width" value="0.1" /> <!-- Square dimensions (widthxwidth) of beams -->
-  <xacro:property name="height1" value="2" /> <!-- Link 1 -->
-  <xacro:property name="height2" value="1" /> <!-- Link 2 -->
-  <xacro:property name="height3" value="1" /> <!-- Link 3 -->
-  <xacro:property name="axel_offset" value="0.05" /> <!-- Space btw top of beam and the each joint -->
-  <joint name="${prefix}base_joint" type="fixed">
-    <xacro:insert_block name="origin" />
-    <parent link="${parent}"/>
-    <child link="${prefix}base_link" />
-  </joint>
-  <!-- Base Link -->
-  <link name="${prefix}base_link">
-    <collision>
-      <origin xyz="0 0 ${height1/2}" rpy="0 0 0"/>
-      <geometry>
-        <box size="${width} ${width} ${height1}"/>
-      </geometry>
-    </collision>
-    <visual>
-      <origin xyz="0 0 ${height1/2}" rpy="0 0 0"/>
-      <geometry>
-        <box size="${width} ${width} ${height1}"/>
-      </geometry>
-      <material name="orange"/>
-    </visual>
-    <inertial>
-      <origin xyz="0 0 ${height1/2}" rpy="0 0 0"/>
-      <mass value="${mass}"/>
-      <inertia
-        ixx="${mass / 12.0 * (width*width + height1*height1)}" ixy="0.0" ixz="0.0"
-        iyy="${mass / 12.0 * (height1*height1 + width*width)}" iyz="0.0"
-        izz="${mass / 12.0 * (width*width + width*width)}"/>
-    </inertial>
-  </link>
-  <joint name="${prefix}joint1" type="continuous">
-    <parent link="${prefix}base_link"/>
-    <child link="${prefix}link1"/>
-    <origin xyz="0 ${width} ${height1 - axel_offset}" rpy="0 0 0"/>
-    <axis xyz="0 1 0"/>
-    <dynamics damping="0.7"/>
-    <limit effort="100" velocity="1.0"/>
-  </joint>
-  <!-- Middle Link -->
-  <link name="${prefix}link1">
-    <collision>
-      <origin xyz="0 0 ${height2/2 - axel_offset}" rpy="0 0 0"/>
-      <geometry>
-        <box size="${width} ${width} ${height2}"/>
-      </geometry>
-    </collision>
-    <visual>
-      <origin xyz="0 0 ${height2/2 - axel_offset}" rpy="0 0 0"/>
-      <geometry>
-        <box size="${width} ${width} ${height2}"/>
-      </geometry>
-      <material name="yellow"/>
-    </visual>
-    <inertial>
-      <origin xyz="0 0 ${height2/2 - axel_offset}" rpy="0 0 0"/>
-      <mass value="${mass}"/>
-      <inertia
-        ixx="${mass / 12.0 * (width*width + height2*height2)}" ixy="0.0" ixz="0.0"
-        iyy="${mass / 12.0 * (height2*height2 + width*width)}" iyz="0.0"
-        izz="${mass / 12.0 * (width*width + width*width)}"/>
-    </inertial>
-  </link>
-  <joint name="${prefix}joint2" type="continuous">
-    <parent link="${prefix}link1"/>
-    <child link="${prefix}link2"/>
-    <origin xyz="0 ${width} ${height2 - axel_offset*2}" rpy="0 0 0"/>
-    <axis xyz="0 1 0"/>
-    <dynamics damping="0.7"/>
-    <limit effort="100" velocity="1.0"/>
-  </joint>
-  <!-- Top Link -->
-  <link name="${prefix}link2">
-    <collision>
-      <origin xyz="0 0 ${height3/2 - axel_offset}" rpy="0 0 0"/>
-      <geometry>
-        <box size="${width} ${width} ${height3}"/>
-      </geometry>
-    </collision>
-    <visual>
-      <origin xyz="0 0 ${height3/2 - axel_offset}" rpy="0 0 0"/>
-      <geometry>
-        <box size="${width} ${width} ${height3}"/>
-      </geometry>
-      <material name="orange"/>
-    </visual>
-    <inertial>
-      <origin xyz="0 0 ${height3/2 - axel_offset}" rpy="0 0 0"/>
-      <mass value="${mass}"/>
-      <inertia
-        ixx="${mass / 12.0 * (width*width + height3*height3)}" ixy="0.0" ixz="0.0"
-        iyy="${mass / 12.0 * (height3*height3 + width*width)}" iyz="0.0"
-        izz="${mass / 12.0 * (width*width + width*width)}"/>
-    </inertial>
-  </link>
-  <joint name="${prefix}tool_joint" type="fixed">
-    <origin xyz="0 0 1" rpy="0 0 0" />
-    <parent link="${prefix}link2"/>
-    <child link="${prefix}tool_link" />
-  </joint>
-  <!-- Tool Link -->
-  <link name="${prefix}tool_link">
-  </link>
+    <!-- 普通参数（字符串类型）`parent`，`prefix`。 block 参数 `*origin` -->
+    <!-- Constants for robot dimensions -->
+    <xacro:property name="mass" value="1" /> <!-- arbitrary value for mass -->
+    <xacro:property name="width" value="0.1" /> <!-- Square dimensions (widthxwidth) of beams -->
+    <xacro:property name="height1" value="2" /> <!-- Link 1 -->
+    <xacro:property name="height2" value="1" /> <!-- Link 2 -->
+    <xacro:property name="height3" value="1" /> <!-- Link 3 -->
+    <xacro:property name="axel_offset" value="0.05" /> <!-- Space btw top of beam and the each joint -->
+    <joint name="${prefix}base_joint" type="fixed">
+      <!--
+        其他xacro调用此 macro时，*origin（block参数） 会被 insert 到下面的 block
+        <xacro:rrbot parent="world" prefix="robot1_">
+          <origin xyz="1 2 0" rpy="0 0 0"/>
+        </xacro:rrbot>
+     -->
+      <xacro:insert_block name="origin" />
+      <parent link="${parent}" />
+      <child link="${prefix}base_link" />
+    </joint>
+    <!-- Base Link -->
+    <link name="${prefix}base_link">
+      <collision>
+        <origin xyz="0 0 ${height1/2}" rpy="0 0 0" />
+        <geometry>
+          <box size="${width} ${width} ${height1}" />
+        </geometry>
+      </collision>
+      <visual>
+        <origin xyz="0 0 ${height1/2}" rpy="0 0 0" />
+        <geometry>
+          <box size="${width} ${width} ${height1}" />
+        </geometry>
+        <material name="orange" />
+      </visual>
+      <inertial>
+        <origin xyz="0 0 ${height1/2}" rpy="0 0 0" />
+        <mass value="${mass}" />
+        <inertia
+          ixx="${mass / 12.0 * (width*width + height1*height1)}" ixy="0.0" ixz="0.0"
+          iyy="${mass / 12.0 * (height1*height1 + width*width)}" iyz="0.0"
+          izz="${mass / 12.0 * (width*width + width*width)}" />
+      </inertial>
+    </link>
+    <joint name="${prefix}joint1" type="continuous">
+      <parent link="${prefix}base_link" />
+      <child link="${prefix}link1" />
+      <origin xyz="0 ${width} ${height1 - axel_offset}" rpy="0 0 0" />
+      <axis xyz="0 1 0" />
+      <dynamics damping="0.7" />
+      <limit effort="100" velocity="1.0" />
+    </joint>
+    <!-- Middle Link -->
+    <link name="${prefix}link1">
+      <collision>
+        <origin xyz="0 0 ${height2/2 - axel_offset}" rpy="0 0 0" />
+        <geometry>
+          <box size="${width} ${width} ${height2}" />
+        </geometry>
+      </collision>
+      <visual>
+        <origin xyz="0 0 ${height2/2 - axel_offset}" rpy="0 0 0" />
+        <geometry>
+          <box size="${width} ${width} ${height2}" />
+        </geometry>
+        <material name="yellow" />
+      </visual>
+      <inertial>
+        <origin xyz="0 0 ${height2/2 - axel_offset}" rpy="0 0 0" />
+        <mass value="${mass}" />
+        <inertia
+          ixx="${mass / 12.0 * (width*width + height2*height2)}" ixy="0.0" ixz="0.0"
+          iyy="${mass / 12.0 * (height2*height2 + width*width)}" iyz="0.0"
+          izz="${mass / 12.0 * (width*width + width*width)}" />
+      </inertial>
+    </link>
+    <joint name="${prefix}joint2" type="continuous">
+      <parent link="${prefix}link1" />
+      <child link="${prefix}link2" />
+      <origin xyz="0 ${width} ${height2 - axel_offset*2}" rpy="0 0 0" />
+      <axis xyz="0 1 0" />
+      <dynamics damping="0.7" />
+      <limit effort="100" velocity="1.0" />
+    </joint>
+    <!-- Top Link -->
+    <link name="${prefix}link2">
+      <collision>
+        <origin xyz="0 0 ${height3/2 - axel_offset}" rpy="0 0 0" />
+        <geometry>
+          <box size="${width} ${width} ${height3}" />
+        </geometry>
+      </collision>
+      <visual>
+        <origin xyz="0 0 ${height3/2 - axel_offset}" rpy="0 0 0" />
+        <geometry>
+          <box size="${width} ${width} ${height3}" />
+        </geometry>
+        <material name="orange" />
+      </visual>
+      <inertial>
+        <origin xyz="0 0 ${height3/2 - axel_offset}" rpy="0 0 0" />
+        <mass value="${mass}" />
+        <inertia
+          ixx="${mass / 12.0 * (width*width + height3*height3)}" ixy="0.0" ixz="0.0"
+          iyy="${mass / 12.0 * (height3*height3 + width*width)}" iyz="0.0"
+          izz="${mass / 12.0 * (width*width + width*width)}" />
+      </inertial>
+    </link>
+    <joint name="${prefix}tool_joint" type="fixed">
+      <origin xyz="0 0 1" rpy="0 0 0" />
+      <parent link="${prefix}link2" />
+      <child link="${prefix}tool_link" />
+    </joint>
+    <!-- Tool Link -->
+    <link name="${prefix}tool_link">
+    </link>
   </xacro:macro>
 </robot>
