Commit message: moveit2案例

File: src/diffbot_gazebo/urdf/gz/diffbot.gazebo.xacro (robot description, xacro)
@@ -3,17 +3,17 @@
 <robot name="diffbot" xmlns:xacro="http://www.ros.org/wiki/xacro">
   <xacro:property name="M_PI" value="3.1415926535897931" />
-  <xacro:property name="d435_cam_width" value="0.090"/>
-  <xacro:property name="d435_cam_height" value="0.025"/>
-  <xacro:property name="d435_cam_depth" value="0.02505"/>
-  <xacro:property name="d435_cam_depth_to_infra1_offset" value="0.0"/>
-  <xacro:property name="d435_cam_depth_to_infra2_offset" value="-0.050"/>
-  <xacro:property name="d435_cam_depth_to_color_offset" value="0.015"/>
-  <xacro:property name="camera_tilt_angle_deg" value="5"/>
+  <xacro:property name="d435_cam_width" value="0.090" />
+  <xacro:property name="d435_cam_height" value="0.025" />
+  <xacro:property name="d435_cam_depth" value="0.02505" />
+  <xacro:property name="d435_cam_depth_to_infra1_offset" value="0.0" />
+  <xacro:property name="d435_cam_depth_to_infra2_offset" value="-0.050" />
+  <xacro:property name="d435_cam_depth_to_color_offset" value="0.015" />
+  <xacro:property name="camera_tilt_angle_deg" value="5" />
   <joint name="camera_depth_joint" type="fixed">
-    <origin xyz="0 0 0" rpy="0 0 0"/>
-    <parent link="camera_link"/>
+    <origin xyz="0 0 0" rpy="0 0 0" />
+    <parent link="camera_link" />
     <child link="camera_depth_frame" />
   </joint>
-  <link name="camera_depth_frame"/>
+  <link name="camera_depth_frame" />
   <joint name="camera_depth_optical_joint" type="fixed">
     <origin xyz="0 0 0" rpy="${-M_PI/2} 0 ${-M_PI/2}" />
@@ -21,5 +21,5 @@
     <child link="camera_depth_optical_frame" />
   </joint>
-  <link name="camera_depth_optical_frame"/>
+  <link name="camera_depth_optical_frame" />
   <joint name="camera_infra1_joint" type="fixed">
     <origin xyz="0 ${d435_cam_depth_to_infra1_offset} 0" rpy="0 0 0" />
@@ -27,5 +27,5 @@
     <child link="camera_infra1_frame" />
   </joint>
-  <link name="camera_infra1_frame"/>
+  <link name="camera_infra1_frame" />
   <joint name="camera_infra1_optical_joint" type="fixed">
     <origin xyz="0 0 0" rpy="${-M_PI/2} 0 ${-M_PI/2}" />
@@ -33,5 +33,5 @@
     <child link="camera_infra1_optical_frame" />
   </joint>
-  <link name="camera_infra1_optical_frame"/>
+  <link name="camera_infra1_optical_frame" />
   <joint name="camera_infra2_joint" type="fixed">
     <origin xyz="0 ${d435_cam_depth_to_infra2_offset} 0" rpy="0 0 0" />
@@ -39,5 +39,5 @@
     <child link="camera_infra2_frame" />
   </joint>
-  <link name="camera_infra2_frame"/>
+  <link name="camera_infra2_frame" />
   <joint name="camera_infra2_optical_joint" type="fixed">
     <origin xyz="0 0 0" rpy="${-M_PI/2} 0 ${-M_PI/2}" />
@@ -45,5 +45,5 @@
     <child link="camera_infra2_optical_frame" />
   </joint>
-  <link name="camera_infra2_optical_frame"/>
+  <link name="camera_infra2_optical_frame" />
   <joint name="camera_color_joint" type="fixed">
     <origin xyz="0 ${d435_cam_depth_to_color_offset} 0" rpy="0 0 0" />
@@ -51,5 +51,5 @@
     <child link="camera_color_frame" />
   </joint>
-  <link name="camera_color_frame"/>
+  <link name="camera_color_frame" />
   <joint name="camera_color_optical_joint" type="fixed">
     <origin xyz="0 0 0" rpy="${-M_PI/2} 0 ${-M_PI/2}" />
@@ -57,6 +57,26 @@
     <child link="camera_color_optical_frame" />
   </joint>
-  <link name="camera_color_optical_frame"/>
-   <gazebo reference="camera_link">
+  <link name="camera_color_optical_frame" />
+  <gazebo reference="caster">
+    <collision>
+      <surface>
+        <friction>
+          <ode>
+            <mu>1</mu>
+            <mu2>1</mu2>
+            <slip1>0.035</slip1>
+            <slip2>0</slip2>
+            <fdir1>0 0 1</fdir1>
+          </ode>
+          <bullet>
+            <friction>1</friction>
+            <friction2>1</friction2>
+            <rolling_friction>0.1</rolling_friction>
+          </bullet>
+        </friction>
+      </surface>
+    </collision>
+  </gazebo>
+  <gazebo reference="camera_link">
     <sensor name="camera" type="rgbd_camera">
       <camera>
@@ -78,126 +98,104 @@
     </sensor>
   </gazebo>
-      <gazebo reference="lidar">
-        <sensor name='gpu_lidar' type='gpu_lidar'>
-          <pose>0 0 0 0 0 0</pose>
-          <topic>scan</topic>
-          <gz_frame_id>lidar</gz_frame_id>
-          <update_rate>10</update_rate>
-          <lidar>
-            <scan>
-              <horizontal>
-                <samples>640</samples>
-                <resolution>1</resolution>
-                <min_angle>-1.396263</min_angle>
-                <max_angle>1.396263</max_angle>
-              </horizontal>
-              <vertical>
-                <samples>1</samples>
-                <resolution>1</resolution>
-                <min_angle>0.0</min_angle>
-                <max_angle>0.0</max_angle>
-              </vertical>
-            </scan>
-            <range>
-              <min>0.08</min>
-              <max>10.0</max>
-              <resolution>0.01</resolution>
-            </range>
-          </lidar>
-          <visualize>true</visualize>
-        </sensor>
-      </gazebo>
+  <gazebo reference="lidar">
+    <sensor name='gpu_lidar' type='gpu_lidar'>
+      <pose>0 0 0 0 0 0</pose>
+      <topic>scan</topic>
+      <gz_frame_id>lidar</gz_frame_id>
+      <update_rate>10</update_rate>
+      <lidar>
+        <scan>
+          <horizontal>
+            <samples>640</samples>
+            <resolution>1</resolution>
+            <min_angle>-1.396263</min_angle>
+            <max_angle>1.396263</max_angle>
+          </horizontal>
+          <vertical>
+            <samples>1</samples>
+            <resolution>1</resolution>
+            <min_angle>0.0</min_angle>
+            <max_angle>0.0</max_angle>
+          </vertical>
+        </scan>
+        <range>
+          <min>0.08</min>
+          <max>10.0</max>
+          <resolution>0.01</resolution>
+        </range>
+      </lidar>
+      <visualize>true</visualize>
+    </sensor>
+  </gazebo>
+  <gazebo reference="imu">
+    <sensor name="imu_sensor" type="imu">
+      <always_on>1</always_on>
+      <update_rate>1</update_rate>
+      <gz_frame_id>imu</gz_frame_id>
+      <visualize>true</visualize>
+      <topic>imu</topic>
+    </sensor>
+  </gazebo>
+  <gazebo reference="left_wheel">
+    <collision>
+      <surface>
+        <friction>
+          <ode>
+            <mu>1</mu>
+            <mu2>1</mu2>
+            <slip1>0.035</slip1>
+            <slip2>0</slip2>
+            <fdir1>0 0 1</fdir1>
+          </ode>
+          <bullet>
+            <friction>1</friction>
+            <friction2>1</friction2>
+            <rolling_friction>0.1</rolling_friction>
+          </bullet>
+        </friction>
+      </surface>
+    </collision>
+  </gazebo>
+  <gazebo reference="right_wheel">
+    <collision>
+      <surface>
+        <friction>
+          <ode>
+            <mu>1</mu>
+            <mu2>1</mu2>
+            <slip1>0.035</slip1>
+            <slip2>0</slip2>
+            <fdir1>0 0 1</fdir1>
+          </ode>
+          <bullet>
+            <friction>1</friction>
+            <friction2>1</friction2>
+            <rolling_friction>0.1</rolling_friction>
+          </bullet>
+        </friction>
+      </surface>
+    </collision>
+  </gazebo>
   <gazebo>
-        <plugin filename="gz-sim-sensors-system" name="gz::sim::systems::Sensors">
-            <render_engine>ogre2</render_engine>
-        </plugin>
-        <plugin filename="gz-sim-imu-system" name="gz::sim::systems::Imu">
-        </plugin>
-        <plugin filename="gz-sim-joint-state-publisher-system" name="gz::sim::systems::JointStatePublisher">
-        <topic>/joint_states</topic>
-        </plugin>
-      <plugin
-        filename="gz-sim-diff-drive-system"
-        name="gz::sim::systems::DiffDrive">
-        <left_joint>left_wheel_joint</left_joint>
-        <right_joint>right_wheel_joint</right_joint>
-        <wheel_separation>1.25</wheel_separation>
-        <wheel_radius>0.3</wheel_radius>
-        <odom_publish_frequency>30</odom_publish_frequency>
-        <topic>/cmd_vel</topic>
-        <tf_topic>/tf</tf_topic>
-        <frame_id>odom</frame_id>
-        <odom_topic>odom</odom_topic>
-        <child_frame_id>base_footprint</child_frame_id>
-</plugin>
- </gazebo>
-    <gazebo reference="imu">
-        <sensor name="imu_sensor" type="imu">
-            <always_on>1</always_on>
-            <update_rate>1</update_rate>
-            <gz_frame_id>imu</gz_frame_id>
-            <visualize>true</visualize>
-            <topic>imu</topic>
-        </sensor>
-    </gazebo>
-   <gazebo reference="left_wheel">
-      <collision>
-        <surface>
-          <friction>
-            <ode>
-              <mu>1</mu>
-              <mu2>1</mu2>
-              <slip1>0.035</slip1>
-              <slip2>0</slip2>
-              <fdir1>0 0 1</fdir1>
-            </ode>
-            <bullet>
-              <friction>1</friction>
-              <friction2>1</friction2>
-              <rolling_friction>0.1</rolling_friction>
-            </bullet>
-          </friction>
-        </surface>
-      </collision>
-  </gazebo>
-   <gazebo reference="right_wheel">
-      <collision>
-        <surface>
-          <friction>
-            <ode>
-              <mu>1</mu>
-              <mu2>1</mu2>
-              <slip1>0.035</slip1>
-              <slip2>0</slip2>
-              <fdir1>0 0 1</fdir1>
-            </ode>
-            <bullet>
-              <friction>1</friction>
-              <friction2>1</friction2>
-              <rolling_friction>0.1</rolling_friction>
-            </bullet>
-          </friction>
-        </surface>
-      </collision>
-  </gazebo>
-   <gazebo reference="caster">
-      <collision>
-        <surface>
-          <friction>
-            <ode>
-              <mu>1</mu>
-              <mu2>1</mu2>
-              <slip1>0.035</slip1>
-              <slip2>0</slip2>
-              <fdir1>0 0 1</fdir1>
-            </ode>
-            <bullet>
-              <friction>1</friction>
-              <friction2>1</friction2>
-              <rolling_friction>0.1</rolling_friction>
-            </bullet>
-          </friction>
-        </surface>
-      </collision>
- </gazebo>
+    <plugin filename="gz-sim-sensors-system" name="gz::sim::systems::Sensors">
+      <render_engine>ogre2</render_engine>
+    </plugin>
+    <plugin filename="gz-sim-imu-system" name="gz::sim::systems::Imu">
+    </plugin>
+    <plugin filename="gz-sim-joint-state-publisher-system" name="gz::sim::systems::JointStatePublisher">
+      <topic>/joint_states</topic>
+    </plugin>
+    <plugin filename="gz-sim-diff-drive-system" name="gz::sim::systems::DiffDrive">
+      <left_joint>left_wheel_joint</left_joint>
+      <right_joint>right_wheel_joint</right_joint>
+      <wheel_separation>1.25</wheel_separation>
+      <wheel_radius>0.3</wheel_radius>
+      <odom_publish_frequency>30</odom_publish_frequency>
+      <topic>/cmd_vel</topic>
+      <tf_topic>/tf</tf_topic>
+      <frame_id>odom</frame_id>
+      <odom_topic>odom</odom_topic>
+      <child_frame_id>base_footprint</child_frame_id>
+    </plugin>
+  </gazebo>
 </robot>
