Commit message: moveit2案例

File: src/diffbot_gazebo/urdf/ros2_control/diffbot.gazebo.xacro (robot description, xacro)
@@ -3,17 +3,17 @@
 <robot name="diffbot" xmlns:xacro="http://www.ros.org/wiki/xacro">
   <xacro:property name="M_PI" value="3.1415926535897931" />
-  <xacro:property name="d435_cam_width" value="0.090"/>
-  <xacro:property name="d435_cam_height" value="0.025"/>
-  <xacro:property name="d435_cam_depth" value="0.02505"/>
-  <xacro:property name="d435_cam_depth_to_infra1_offset" value="0.0"/>
-  <xacro:property name="d435_cam_depth_to_infra2_offset" value="-0.050"/>
-  <xacro:property name="d435_cam_depth_to_color_offset" value="0.015"/>
-  <xacro:property name="camera_tilt_angle_deg" value="5"/>
+  <xacro:property name="d435_cam_width" value="0.090" />
+  <xacro:property name="d435_cam_height" value="0.025" />
+  <xacro:property name="d435_cam_depth" value="0.02505" />
+  <xacro:property name="d435_cam_depth_to_infra1_offset" value="0.0" />
+  <xacro:property name="d435_cam_depth_to_infra2_offset" value="-0.050" />
+  <xacro:property name="d435_cam_depth_to_color_offset" value="0.015" />
+  <xacro:property name="camera_tilt_angle_deg" value="5" />
   <joint name="camera_depth_joint" type="fixed">
-    <origin xyz="0 0 0" rpy="0 0 0"/>
-    <parent link="camera_link"/>
+    <origin xyz="0 0 0" rpy="0 0 0" />
+    <parent link="camera_link" />
     <child link="camera_depth_frame" />
   </joint>
-  <link name="camera_depth_frame"/>
+  <link name="camera_depth_frame" />
   <joint name="camera_depth_optical_joint" type="fixed">
     <origin xyz="0 0 0" rpy="${-M_PI/2} 0 ${-M_PI/2}" />
@@ -21,5 +21,5 @@
     <child link="camera_depth_optical_frame" />
   </joint>
-  <link name="camera_depth_optical_frame"/>
+  <link name="camera_depth_optical_frame" />
   <joint name="camera_infra1_joint" type="fixed">
     <origin xyz="0 ${d435_cam_depth_to_infra1_offset} 0" rpy="0 0 0" />
@@ -27,5 +27,5 @@
     <child link="camera_infra1_frame" />
   </joint>
-  <link name="camera_infra1_frame"/>
+  <link name="camera_infra1_frame" />
   <joint name="camera_infra1_optical_joint" type="fixed">
     <origin xyz="0 0 0" rpy="${-M_PI/2} 0 ${-M_PI/2}" />
@@ -33,5 +33,5 @@
     <child link="camera_infra1_optical_frame" />
   </joint>
-  <link name="camera_infra1_optical_frame"/>
+  <link name="camera_infra1_optical_frame" />
   <joint name="camera_infra2_joint" type="fixed">
     <origin xyz="0 ${d435_cam_depth_to_infra2_offset} 0" rpy="0 0 0" />
@@ -39,5 +39,5 @@
     <child link="camera_infra2_frame" />
   </joint>
-  <link name="camera_infra2_frame"/>
+  <link name="camera_infra2_frame" />
   <joint name="camera_infra2_optical_joint" type="fixed">
     <origin xyz="0 0 0" rpy="${-M_PI/2} 0 ${-M_PI/2}" />
@@ -45,5 +45,5 @@
     <child link="camera_infra2_optical_frame" />
   </joint>
-  <link name="camera_infra2_optical_frame"/>
+  <link name="camera_infra2_optical_frame" />
   <joint name="camera_color_joint" type="fixed">
     <origin xyz="0 ${d435_cam_depth_to_color_offset} 0" rpy="0 0 0" />
@@ -51,5 +51,5 @@
     <child link="camera_color_frame" />
   </joint>
-  <link name="camera_color_frame"/>
+  <link name="camera_color_frame" />
   <joint name="camera_color_optical_joint" type="fixed">
     <origin xyz="0 0 0" rpy="${-M_PI/2} 0 ${-M_PI/2}" />
@@ -57,6 +57,6 @@
     <child link="camera_color_optical_frame" />
   </joint>
-  <link name="camera_color_optical_frame"/>
-   <gazebo reference="camera_link">
+  <link name="camera_color_optical_frame" />
+  <gazebo reference="camera_link">
     <sensor name="camera" type="rgbd_camera">
       <camera>
@@ -78,141 +78,141 @@
     </sensor>
   </gazebo>
-      <gazebo reference="lidar">
-        <sensor name='gpu_lidar' type='gpu_lidar'>
-          <pose>0 0 0 0 0 0</pose>
-          <topic>scan</topic>
-          <gz_frame_id>lidar</gz_frame_id>
-          <update_rate>10</update_rate>
-          <lidar>
-            <scan>
-              <horizontal>
-                <samples>640</samples>
-                <resolution>1</resolution>
-                <min_angle>-1.396263</min_angle>
-                <max_angle>1.396263</max_angle>
-              </horizontal>
-              <vertical>
-                <samples>1</samples>
-                <resolution>1</resolution>
-                <min_angle>0.0</min_angle>
-                <max_angle>0.0</max_angle>
-              </vertical>
-            </scan>
-            <range>
-              <min>0.08</min>
-              <max>10.0</max>
-              <resolution>0.01</resolution>
-            </range>
-          </lidar>
-          <visualize>true</visualize>
-        </sensor>
-      </gazebo>
+  <gazebo reference="lidar">
+    <sensor name='gpu_lidar' type='gpu_lidar'>
+      <pose>0 0 0 0 0 0</pose>
+      <topic>scan</topic>
+      <gz_frame_id>lidar</gz_frame_id>
+      <update_rate>10</update_rate>
+      <lidar>
+        <scan>
+          <horizontal>
+            <samples>640</samples>
+            <resolution>1</resolution>
+            <min_angle>-1.396263</min_angle>
+            <max_angle>1.396263</max_angle>
+          </horizontal>
+          <vertical>
+            <samples>1</samples>
+            <resolution>1</resolution>
+            <min_angle>0.0</min_angle>
+            <max_angle>0.0</max_angle>
+          </vertical>
+        </scan>
+        <range>
+          <min>0.08</min>
+          <max>10.0</max>
+          <resolution>0.01</resolution>
+        </range>
+      </lidar>
+      <visualize>true</visualize>
+    </sensor>
+  </gazebo>
   <gazebo>
-        <plugin filename="gz-sim-sensors-system" name="gz::sim::systems::Sensors">
-            <render_engine>ogre2</render_engine>
-        </plugin>
-        <plugin filename="gz-sim-imu-system" name="gz::sim::systems::Imu">
-        </plugin>
- <!--
-        <plugin filename="gz-sim-joint-state-publisher-system" name="gz::sim::systems::JointStatePublisher">
-        </plugin>
-      <plugin
-        filename="gz-sim-diff-drive-system"
-        name="gz::sim::systems::DiffDrive">
-        <left_joint>left_wheel_joint</left_joint>
-        <right_joint>right_wheel_joint</right_joint>
-        <wheel_separation>1.25</wheel_separation>
-        <wheel_radius>0.3</wheel_radius>
-        <odom_publish_frequency>30</odom_publish_frequency>
-        <topic>/cmd_vel</topic>
-        <tf_topic>/tf</tf_topic>
-        <frame_id>odom</frame_id>
-        <child_frame_id>base_link</child_frame_id>
-        <max_linear_acceleration>1</max_linear_acceleration>
-        <min_linear_acceleration>-1</min_linear_acceleration>
-        <max_angular_acceleration>2</max_angular_acceleration>
-        <min_angular_acceleration>-2</min_angular_acceleration>
-        <max_linear_velocity>0.5</max_linear_velocity>
-        <min_linear_velocity>-0.5</min_linear_velocity>
-        <max_angular_velocity>1</max_angular_velocity>
-        <min_angular_velocity>-1</min_angular_velocity>
-      </plugin>
--->
-  <!-- Gazebo ROS 2 Control plugin -->
-        <plugin filename="gz_ros2_control-system" name="gz_ros2_control::GazeboSimROS2ControlPlugin">
-            <parameters>$(find diffbot_gazebo)/config/diffbot_controllers.yaml</parameters>
-            <ros>
-                <remapping>/controller_manager/robot_description:=/robot_description</remapping>
-            </ros>
-        </plugin>
-  </gazebo>
-    <gazebo reference="imu">
-        <sensor name="imu_sensor" type="imu">
-            <always_on>1</always_on>
-            <update_rate>1</update_rate>
-            <gz_frame_id>imu</gz_frame_id>
-            <visualize>true</visualize>
-            <topic>imu</topic>
-        </sensor>
-    </gazebo>
-   <gazebo reference="left_wheel">
-      <collision>
-        <surface>
-          <friction>
-            <ode>
-              <mu>1</mu>
-              <mu2>1</mu2>
-              <slip1>0.035</slip1>
-              <slip2>0</slip2>
-              <fdir1>0 0 1</fdir1>
-            </ode>
-            <bullet>
-              <friction>1</friction>
-              <friction2>1</friction2>
-              <rolling_friction>0.1</rolling_friction>
-            </bullet>
-          </friction>
-        </surface>
-      </collision>
-  </gazebo>
-   <gazebo reference="right_wheel">
-      <collision>
-        <surface>
-          <friction>
-            <ode>
-              <mu>1</mu>
-              <mu2>1</mu2>
-              <slip1>0.035</slip1>
-              <slip2>0</slip2>
-              <fdir1>0 0 1</fdir1>
-            </ode>
-            <bullet>
-              <friction>1</friction>
-              <friction2>1</friction2>
-              <rolling_friction>0.1</rolling_friction>
-            </bullet>
-          </friction>
-        </surface>
-      </collision>
-  </gazebo>
-   <gazebo reference="caster">
-      <collision>
-        <surface>
-          <friction>
-            <ode>
-              <mu>1</mu>
-              <mu2>1</mu2>
-              <slip1>0.035</slip1>
-              <slip2>0</slip2>
-              <fdir1>0 0 1</fdir1>
-            </ode>
-            <bullet>
-              <friction>1</friction>
-              <friction2>1</friction2>
-              <rolling_friction>0.1</rolling_friction>
-            </bullet>
-          </friction>
-        </surface>
-      </collision>
- </gazebo>
+    <plugin filename="gz-sim-sensors-system" name="gz::sim::systems::Sensors">
+      <render_engine>ogre2</render_engine>
+    </plugin>
+    <plugin filename="gz-sim-imu-system" name="gz::sim::systems::Imu">
+    </plugin>
+    <!-- 使用GZ-SIM Plugin 要用到的插件，放在这里方便和ROS2Control做对比 -->
+    <!-- <plugin filename="gz-sim-joint-state-publisher-system"
+      name="gz::sim::systems::JointStatePublisher">
+    </plugin>
+    <plugin
+      filename="gz-sim-diff-drive-system"
+      name="gz::sim::systems::DiffDrive">
+      <left_joint>left_wheel_joint</left_joint>
+      <right_joint>right_wheel_joint</right_joint>
+      <wheel_separation>1.25</wheel_separation>
+      <wheel_radius>0.3</wheel_radius>
+      <odom_publish_frequency>30</odom_publish_frequency>
+      <topic>/cmd_vel</topic>
+      <tf_topic>/tf</tf_topic>
+      <frame_id>odom</frame_id>
+      <child_frame_id>base_link</child_frame_id>
+      <max_linear_acceleration>1</max_linear_acceleration>
+      <min_linear_acceleration>-1</min_linear_acceleration>
+      <max_angular_acceleration>2</max_angular_acceleration>
+      <min_angular_acceleration>-2</min_angular_acceleration>
+      <max_linear_velocity>0.5</max_linear_velocity>
+      <min_linear_velocity>-0.5</min_linear_velocity>
+      <max_angular_velocity>1</max_angular_velocity>
+      <min_angular_velocity>-1</min_angular_velocity>
+    </plugin> -->
+    <!-- Gazebo ROS 2 Control plugin -->
+    <plugin filename="gz_ros2_control-system" name="gz_ros2_control::GazeboSimROS2ControlPlugin">
+      <parameters>$(find diffbot_gazebo)/config/diffbot_controllers.yaml</parameters>
+      <ros>
+        <remapping>/controller_manager/robot_description:=/robot_description</remapping>
+      </ros>
+    </plugin>
+  </gazebo>
+  <gazebo reference="imu">
+    <sensor name="imu_sensor" type="imu">
+      <always_on>1</always_on>
+      <update_rate>1</update_rate>
+      <gz_frame_id>imu</gz_frame_id>
+      <visualize>true</visualize>
+      <topic>imu</topic>
+    </sensor>
+  </gazebo>
+  <gazebo reference="left_wheel">
+    <collision>
+      <surface>
+        <friction>
+          <ode>
+            <mu>1</mu>
+            <mu2>1</mu2>
+            <slip1>0.035</slip1>
+            <slip2>0</slip2>
+            <fdir1>0 0 1</fdir1>
+          </ode>
+          <bullet>
+            <friction>1</friction>
+            <friction2>1</friction2>
+            <rolling_friction>0.1</rolling_friction>
+          </bullet>
+        </friction>
+      </surface>
+    </collision>
+  </gazebo>
+  <gazebo reference="right_wheel">
+    <collision>
+      <surface>
+        <friction>
+          <ode>
+            <mu>1</mu>
+            <mu2>1</mu2>
+            <slip1>0.035</slip1>
+            <slip2>0</slip2>
+            <fdir1>0 0 1</fdir1>
+          </ode>
+          <bullet>
+            <friction>1</friction>
+            <friction2>1</friction2>
+            <rolling_friction>0.1</rolling_friction>
+          </bullet>
+        </friction>
+      </surface>
+    </collision>
+  </gazebo>
+  <gazebo reference="caster">
+    <collision>
+      <surface>
+        <friction>
+          <ode>
+            <mu>1</mu>
+            <mu2>1</mu2>
+            <slip1>0.035</slip1>
+            <slip2>0</slip2>
+            <fdir1>0 0 1</fdir1>
+          </ode>
+          <bullet>
+            <friction>1</friction>
+            <friction2>1</friction2>
+            <rolling_friction>0.1</rolling_friction>
+          </bullet>
+        </friction>
+      </surface>
+    </collision>
+  </gazebo>
 </robot>

File: src/diffbot_gazebo/urdf/ros2_control/diffbot.xacro (robot description, xacro)
@@ -2,30 +2,30 @@
 <!-- Revolute-Revolute Manipulator -->
 <robot name="diffbot" xmlns:xacro="http://www.ros.org/wiki/xacro">
-  <xacro:include filename="$(find diffbot_gazebo)/urdf/ros2_control/diffbot.gazebo.xacro"/>
-  <xacro:include filename="$(find diffbot_gazebo)/urdf/ros2_control/diffbot.ros2_control.xacro"/>
+  <xacro:include filename="$(find diffbot_gazebo)/urdf/ros2_control/diffbot.gazebo.xacro" />
+  <xacro:include filename="$(find diffbot_gazebo)/urdf/ros2_control/diffbot.ros2_control.xacro" />
   <!-- Chassis -->
-  <link name="base_footprint"/>
-    <joint name="base_joint" type="fixed">
-        <parent link="base_footprint"/>
-        <child link="base_link"/>
-        <origin xyz="0.0 0 0" rpy="0 0 0.0" />
-    </joint>
+  <link name="base_footprint" />
+  <joint name="base_joint" type="fixed">
+    <parent link="base_footprint" />
+    <child link="base_link" />
+    <origin xyz="0.0 0 0" rpy="0 0 0.0" />
+  </joint>
   <link name="base_link">
     <visual>
       <geometry>
-        <box size="2.0 1.0 0.5"/>
+        <box size="2.0 1.0 0.5" />
       </geometry>
       <material name="blue">
-        <color rgba="0.0 0.0 1.0 1"/>
+        <color rgba="0.0 0.0 1.0 1" />
       </material>
     </visual>
     <collision>
       <geometry>
-        <box size="2.0 1.0 0.5"/>
+        <box size="2.0 1.0 0.5" />
       </geometry>
     </collision>
     <inertial>
-      <mass value="1.14395"/>
-      <inertia ixx="0.126164" ixy="0" ixz="0" iyy="0.416519" iyz="0" izz="0.481014"/>
+      <mass value="1.14395" />
+      <inertia ixx="0.126164" ixy="0" ixz="0" iyy="0.416519" iyz="0" izz="0.481014" />
     </inertial>
   </link>
@@ -34,18 +34,18 @@
     <visual>
       <geometry>
-        <cylinder radius="0.4" length="0.2"/>
+        <cylinder radius="0.4" length="0.2" />
       </geometry>
       <material name="red">
-        <color rgba="1.0 0.0 0.0 1"/>
+        <color rgba="1.0 0.0 0.0 1" />
       </material>
     </visual>
     <collision>
       <geometry>
-        <cylinder radius="0.4" length="0.2"/>
+        <cylinder radius="0.4" length="0.2" />
       </geometry>
     </collision>
     <inertial>
-      <mass value="2.0"/>
-      <inertia ixx="0.145833" ixy="0" ixz="0" iyy="0.145833" iyz="0" izz="0.125"/>
+      <mass value="2.0" />
+      <inertia ixx="0.145833" ixy="0" ixz="0" iyy="0.145833" iyz="0" izz="0.125" />
     </inertial>
   </link>
@@ -54,18 +54,18 @@
     <visual>
       <geometry>
-        <cylinder radius="0.4" length="0.2"/>
+        <cylinder radius="0.4" length="0.2" />
       </geometry>
       <material name="red">
-        <color rgba="1.0 0.0 0.0 1"/>
+        <color rgba="1.0 0.0 0.0 1" />
       </material>
     </visual>
     <collision>
       <geometry>
-        <cylinder radius="0.4" length="0.2"/>
+        <cylinder radius="0.4" length="0.2" />
       </geometry>
     </collision>
     <inertial>
-      <mass value="1.0"/>
-      <inertia ixx="0.145833" ixy="0" ixz="0" iyy="0.145833" iyz="0" izz="0.125"/>
+      <mass value="1.0" />
+      <inertia ixx="0.145833" ixy="0" ixz="0" iyy="0.145833" iyz="0" izz="0.125" />
     </inertial>
   </link>
@@ -74,18 +74,18 @@
     <visual>
       <geometry>
-        <sphere radius="0.2"/>
+        <sphere radius="0.2" />
       </geometry>
       <material name="green">
-        <color rgba="0.0 1.0 0.0 1"/>
+        <color rgba="0.0 1.0 0.0 1" />
       </material>
     </visual>
     <collision>
       <geometry>
-        <sphere radius="0.2"/>
+        <sphere radius="0.2" />
       </geometry>
     </collision>
     <inertial>
-      <mass value="1.0"/>
-      <inertia ixx="0.1" ixy="0" ixz="0" iyy="0.1" iyz="0" izz="0.1"/>
+      <mass value="1.0" />
+      <inertia ixx="0.1" ixy="0" ixz="0" iyy="0.1" iyz="0" izz="0.1" />
     </inertial>
   </link>
@@ -94,18 +94,18 @@
     <visual>
       <geometry>
-        <box size="0.2 0.2 0.2"/>
+        <box size="0.2 0.2 0.2" />
       </geometry>
       <material name="green">
-        <color rgba="0.0 1.0 0.0 1"/>
+        <color rgba="0.0 1.0 0.0 1" />
       </material>
     </visual>
     <collision>
       <geometry>
-        <box size="0.2 0.2 0.2"/>
+        <box size="0.2 0.2 0.2" />
       </geometry>
     </collision>
     <inertial>
-      <mass value="1.0"/>
-      <inertia ixx="0.1" ixy="0" ixz="0" iyy="0.1" iyz="0" izz="0.1"/>
+      <mass value="1.0" />
+      <inertia ixx="0.1" ixy="0" ixz="0" iyy="0.1" iyz="0" izz="0.1" />
     </inertial>
   </link>
@@ -114,18 +114,18 @@
     <visual>
       <geometry>
-        <box size="0.2 0.2 0.2"/>
+        <box size="0.2 0.2 0.2" />
       </geometry>
       <material name="red">
-        <color rgba="0.0 1.0 0.0 1"/>
+        <color rgba="0.0 1.0 0.0 1" />
       </material>
     </visual>
     <collision>
       <geometry>
-        <box size="0.2 0.2 0.2"/>
+        <box size="0.2 0.2 0.2" />
       </geometry>
     </collision>
     <inertial>
-      <mass value="1.0"/>
-      <inertia ixx="0.1" ixy="0" ixz="0" iyy="0.1" iyz="0" izz="0.1"/>
+      <mass value="1.0" />
+      <inertia ixx="0.1" ixy="0" ixz="0" iyy="0.1" iyz="0" izz="0.1" />
     </inertial>
   </link>
@@ -134,54 +134,54 @@
     <visual>
       <geometry>
-        <box size="0.2 0.2 0.2"/>
+        <box size="0.2 0.2 0.2" />
       </geometry>
       <material name="red">
-        <color rgba="1.0 0.0 1.0 1"/>
+        <color rgba="1.0 0.0 1.0 1" />
       </material>
     </visual>
     <collision>
       <geometry>
-        <box size="0.2 0.2 0.2"/>
+        <box size="0.2 0.2 0.2" />
       </geometry>
     </collision>
     <inertial>
-      <mass value="1.0"/>
-      <inertia ixx="0.1" ixy="0" ixz="0" iyy="0.1" iyz="0" izz="0.1"/>
+      <mass value="1.0" />
+      <inertia ixx="0.1" ixy="0" ixz="0" iyy="0.1" iyz="0" izz="0.1" />
     </inertial>
   </link>
   <!-- Joints -->
   <joint name="left_wheel_joint" type="continuous">
-    <parent link="base_link"/>
-    <child link="left_wheel"/>
-    <origin xyz="-0.5 0.6 0" rpy="-1.5707 0 0"/>
-    <axis xyz="0 0 1"/>
-    <dynamics damping="0.02"/>
+    <parent link="base_link" />
+    <child link="left_wheel" />
+    <origin xyz="-0.5 0.6 0" rpy="-1.5707 0 0" />
+    <axis xyz="0 0 1" />
+    <dynamics damping="0.02" />
   </joint>
   <joint name="right_wheel_joint" type="continuous">
-    <parent link="base_link"/>
-    <child link="right_wheel"/>
-    <origin xyz="-0.5 -0.6 0" rpy="-1.5707 0 0"/>
-    <axis xyz="0 0 1"/>
-    <dynamics damping="0.02"/>
+    <parent link="base_link" />
+    <child link="right_wheel" />
+    <origin xyz="-0.5 -0.6 0" rpy="-1.5707 0 0" />
+    <axis xyz="0 0 1" />
+    <dynamics damping="0.02" />
   </joint>
   <joint name="caster_joint" type="fixed">
-    <parent link="base_link"/>
-    <child link="caster"/>
-    <origin xyz="0.8 0 -0.2" rpy="0 0 0"/>
+    <parent link="base_link" />
+    <child link="caster" />
+    <origin xyz="0.8 0 -0.2" rpy="0 0 0" />
   </joint>
   <joint name="depth_joint" type="fixed">
-    <parent link="base_link"/>
-    <child link="camera_link"/>
-    <origin xyz="0.9 0 0.36" rpy="0 0 0"/>
+    <parent link="base_link" />
+    <child link="camera_link" />
+    <origin xyz="0.9 0 0.36" rpy="0 0 0" />
   </joint>
   <joint name="lidar_joint" type="fixed">
-    <parent link="base_link"/>
-    <child link="lidar"/>
-    <origin xyz="0.9 0 0.56" rpy="0 0 0"/>
+    <parent link="base_link" />
+    <child link="lidar" />
+    <origin xyz="0.9 0 0.56" rpy="0 0 0" />
   </joint>
   <joint name="imu_joint" type="fixed">
-    <parent link="base_link"/>
-    <child link="imu"/>
-    <origin xyz="0.0 0 0.36" rpy="0 0 0"/>
+    <parent link="base_link" />
+    <child link="imu" />
+    <origin xyz="0.0 0 0.36" rpy="0 0 0" />
   </joint>
 </robot>
