Commit message: 注释,优化执行链

File: src/panda_description/urdf/panda_gripper.xacro (robot description, xacro)
@@ -5,49 +5,50 @@
   <!-- Imported elements -->
   <!--                   -->
-  <xacro:include filename="$(find panda_description)/urdf/panda_utils.xacro"/>
+  <xacro:include filename="$(find panda_description)/urdf/panda_utils.xacro" />
   <!--            -->
   <!-- Properties -->
   <!--            -->
-  <xacro:property name="joint_wrist_name" value="joint_wrist"/>
-  <xacro:property name="joint_wrist_type" value="fixed"/>
-  <xacro:property name="hand_name" value="hand"/>
-  <xacro:property name="hand_mu" value="0.85"/>
-  <xacro:property name="joint_finger1_name" value="finger_joint1"/>
-  <xacro:property name="joint_finger1_type" value="prismatic"/>
-  <xacro:property name="joint_finger1_origin_xyz" value="0 0 0.0584"/>
-  <xacro:property name="joint_finger1_origin_rpy" value="0 0 0"/>
-  <xacro:property name="joint_finger1_axis_xyz" value="0 1 0"/>
-  <xacro:property name="joint_finger1_lower_limit" value="0"/>
-  <xacro:property name="joint_finger1_upper_limit" value="0.04"/>
-  <xacro:property name="joint_finger1_velocity_limit" value="0.2"/>
-  <xacro:property name="joint_finger1_torque_limit" value="20"/>
-  <xacro:property name="joint_finger1_damping" value="3.0"/>
-  <xacro:property name="joint_finger1_friction" value="0.4"/>
-  <xacro:property name="link_finger1_name" value="leftfinger"/>
-  <xacro:property name="link_finger1_mu" value="1.13"/>
-  <xacro:property name="link_finger1_mesh_offset" value="0 0 0"/>
-  <xacro:property name="joint_finger2_name" value="finger_joint2"/>
-  <xacro:property name="joint_finger2_type" value="prismatic"/>
-  <xacro:property name="joint_finger2_origin_xyz" value="0 0 0.0584"/>
-  <xacro:property name="joint_finger2_origin_rpy" value="0 0 0"/>
-  <xacro:property name="joint_finger2_axis_xyz" value="0 -1 0"/>
-  <xacro:property name="joint_finger2_lower_limit" value="0"/>
-  <xacro:property name="joint_finger2_upper_limit" value="0.04"/>
-  <xacro:property name="joint_finger2_velocity_limit" value="0.2"/>
-  <xacro:property name="joint_finger2_torque_limit" value="20"/>
-  <xacro:property name="joint_finger2_damping" value="3.0"/>
-  <xacro:property name="joint_finger2_friction" value="0.4"/>
-  <xacro:property name="link_finger2_name" value="rightfinger"/>
-  <xacro:property name="link_finger2_mu" value="1.13"/>
-  <xacro:property name="link_finger2_mesh_offset" value="0 0 ${pi}"/>
-  <xacro:property name="ee_name" value="hand_tcp"/>
-  <xacro:property name="ee_origin_xyz" value="0 0 0.1034"/>
-  <xacro:property name="ee_origin_rpy" value="0 0 0"/>
+  <xacro:property name="joint_wrist_name" value="joint_wrist" />
+  <xacro:property name="joint_wrist_type" value="fixed" />
+  <xacro:property name="hand_name" value="hand" />
+  <xacro:property name="hand_mu" value="0.85" />
+  <xacro:property name="joint_finger1_name" value="finger_joint1" />
+  <xacro:property name="joint_finger1_type" value="prismatic" />
+  <xacro:property name="joint_finger1_origin_xyz" value="0 0 0.0584" />
+  <xacro:property name="joint_finger1_origin_rpy" value="0 0 0" />
+  <xacro:property name="joint_finger1_axis_xyz" value="0 1 0" />
+  <xacro:property name="joint_finger1_lower_limit" value="0" />
+  <xacro:property name="joint_finger1_upper_limit" value="0.04" />
+  <xacro:property name="joint_finger1_velocity_limit" value="0.2" />
+  <xacro:property name="joint_finger1_torque_limit" value="20" />
+  <xacro:property name="joint_finger1_damping" value="3.0" />
+  <xacro:property name="joint_finger1_friction" value="0.4" />
+  <xacro:property name="link_finger1_name" value="leftfinger" />
+  <xacro:property name="link_finger1_mu" value="1.13" />
+  <xacro:property name="link_finger1_mesh_offset" value="0 0 0" />
+  <xacro:property name="joint_finger2_name" value="finger_joint2" />
+  <xacro:property name="joint_finger2_type" value="prismatic" />
+  <xacro:property name="joint_finger2_origin_xyz" value="0 0 0.0584" />
+  <xacro:property name="joint_finger2_origin_rpy" value="0 0 0" />
+  <xacro:property name="joint_finger2_axis_xyz" value="0 -1 0" />
+  <xacro:property name="joint_finger2_lower_limit" value="0" />
+  <xacro:property name="joint_finger2_upper_limit" value="0.04" />
+  <xacro:property name="joint_finger2_velocity_limit" value="0.2" />
+  <xacro:property name="joint_finger2_torque_limit" value="20" />
+  <xacro:property name="joint_finger2_damping" value="3.0" />
+  <xacro:property name="joint_finger2_friction" value="0.4" />
+  <xacro:property name="link_finger2_name" value="rightfinger" />
+  <xacro:property name="link_finger2_mu" value="1.13" />
+  <xacro:property name="link_finger2_mesh_offset" value="0 0 ${pi}" />
+  <xacro:property name="ee_name" value="hand_tcp" />
+  <xacro:property name="ee_origin_xyz" value="0 0 0.1034" />
+  <xacro:property name="ee_origin_rpy" value="0 0 0" />
   <!--       -->
   <!-- Macro -->
   <!--       -->
-  <xacro:property name="default_origin_xyz" value="0 0 0"/>
-  <xacro:property name="default_origin_rpy" value="0 0 0"/>
-  <xacro:macro name="panda_gripper" params="
+  <xacro:property name="default_origin_xyz" value="0 0 0" />
+  <xacro:property name="default_origin_rpy" value="0 0 0" />
+  <xacro:macro name="panda_gripper"
+    params="
     wrist_flange
     prefix:=panda_
@@ -62,73 +63,73 @@
     <!-- Wrist -->
     <xacro:panda_joint
-    parent="${wrist_flange}"
-    child="${prefix}${hand_name}"
-    joint_name="${prefix}${joint_wrist_name}"
-    joint_type="${joint_wrist_type}"
-    joint_origin_xyz="${origin_xyz}"
-    joint_origin_rpy="${origin_rpy}"
-    gazebo_preserve_fixed_joint="${gazebo_preserve_fixed_joint}"
+      parent="${wrist_flange}"
+      child="${prefix}${hand_name}"
+      joint_name="${prefix}${joint_wrist_name}"
+      joint_type="${joint_wrist_type}"
+      joint_origin_xyz="${origin_xyz}"
+      joint_origin_rpy="${origin_rpy}"
+      gazebo_preserve_fixed_joint="${gazebo_preserve_fixed_joint}"
     />
     <xacro:panda_link
-    link_name="${prefix}${hand_name}"
-    mesh="${hand_mesh}"
-    collision="${collision}"
-    mu="${hand_mu}"
+      link_name="${prefix}${hand_name}"
+      mesh="${hand_mesh}"
+      collision="${collision}"
+      mu="${hand_mu}"
     />
     <!-- Finger 1 -->
     <xacro:panda_joint
-    parent="${prefix}${hand_name}"
-    child="${prefix}${link_finger1_name}"
-    joint_name="${prefix}${joint_finger1_name}"
-    joint_type="${joint_finger1_type}"
-    joint_origin_xyz="${joint_finger1_origin_xyz}"
-    joint_origin_rpy="${joint_finger1_origin_rpy}"
-    joint_axis_xyz="${joint_finger1_axis_xyz}"
-    joint_lower_limit="${joint_finger1_lower_limit}"
-    joint_upper_limit="${joint_finger1_upper_limit}"
-    joint_velocity_limit="${joint_finger1_velocity_limit}"
-    joint_torque_limit="${joint_finger1_torque_limit}"
-    joint_damping="${joint_finger1_damping}"
-    joint_friction="${joint_finger1_friction}"
-    gazebo_preserve_fixed_joint="${gazebo_preserve_fixed_joint}"
+      parent="${prefix}${hand_name}"
+      child="${prefix}${link_finger1_name}"
+      joint_name="${prefix}${joint_finger1_name}"
+      joint_type="${joint_finger1_type}"
+      joint_origin_xyz="${joint_finger1_origin_xyz}"
+      joint_origin_rpy="${joint_finger1_origin_rpy}"
+      joint_axis_xyz="${joint_finger1_axis_xyz}"
+      joint_lower_limit="${joint_finger1_lower_limit}"
+      joint_upper_limit="${joint_finger1_upper_limit}"
+      joint_velocity_limit="${joint_finger1_velocity_limit}"
+      joint_torque_limit="${joint_finger1_torque_limit}"
+      joint_damping="${joint_finger1_damping}"
+      joint_friction="${joint_finger1_friction}"
+      gazebo_preserve_fixed_joint="${gazebo_preserve_fixed_joint}"
     />
     <xacro:panda_link
-    link_name="${prefix}${link_finger1_name}"
-    mesh="${finger_mesh}"
-    collision="${collision}"
-    mu="${link_finger1_mu}"
-    mesh_offset_rpy="${link_finger1_mesh_offset}"
+      link_name="${prefix}${link_finger1_name}"
+      mesh="${finger_mesh}"
+      collision="${collision}"
+      mu="${link_finger1_mu}"
+      mesh_offset_rpy="${link_finger1_mesh_offset}"
     />
     <!-- Finger 2 -->
     <xacro:panda_joint
-    parent="${prefix}${hand_name}"
-    child="${prefix}${link_finger2_name}"
-    joint_name="${prefix}${joint_finger2_name}"
-    joint_type="${joint_finger2_type}"
-    joint_origin_xyz="${joint_finger2_origin_xyz}"
-    joint_origin_rpy="${joint_finger2_origin_rpy}"
-    joint_axis_xyz="${joint_finger2_axis_xyz}"
-    joint_lower_limit="${joint_finger2_lower_limit}"
-    joint_upper_limit="${joint_finger2_upper_limit}"
-    joint_velocity_limit="${joint_finger2_velocity_limit}"
-    joint_torque_limit="${joint_finger2_torque_limit}"
-    joint_damping="${joint_finger2_damping}"
-    joint_friction="${joint_finger2_friction}"
-    gazebo_preserve_fixed_joint="${gazebo_preserve_fixed_joint}"
+      parent="${prefix}${hand_name}"
+      child="${prefix}${link_finger2_name}"
+      joint_name="${prefix}${joint_finger2_name}"
+      joint_type="${joint_finger2_type}"
+      joint_origin_xyz="${joint_finger2_origin_xyz}"
+      joint_origin_rpy="${joint_finger2_origin_rpy}"
+      joint_axis_xyz="${joint_finger2_axis_xyz}"
+      joint_lower_limit="${joint_finger2_lower_limit}"
+      joint_upper_limit="${joint_finger2_upper_limit}"
+      joint_velocity_limit="${joint_finger2_velocity_limit}"
+      joint_torque_limit="${joint_finger2_torque_limit}"
+      joint_damping="${joint_finger2_damping}"
+      joint_friction="${joint_finger2_friction}"
+      gazebo_preserve_fixed_joint="${gazebo_preserve_fixed_joint}"
     />
     <xacro:panda_link
-    link_name="${prefix}${link_finger2_name}"
-    mesh="${finger_mesh}"
-    collision="${collision}"
-    mu="${link_finger2_mu}"
-    mesh_offset_rpy="${link_finger2_mesh_offset}"
+      link_name="${prefix}${link_finger2_name}"
+      mesh="${finger_mesh}"
+      collision="${collision}"
+      mu="${link_finger2_mu}"
+      mesh_offset_rpy="${link_finger2_mesh_offset}"
     />
     <!-- End effector -->
     <xacro:panda_virtual_link
-    parent="${prefix}${hand_name}"
-    link_name="${prefix}${ee_name}"
-    joint_origin_xyz="${ee_origin_xyz}"
-    joint_origin_rpy="${ee_origin_rpy}"
-    gazebo_preserve_fixed_joint="${gazebo_preserve_fixed_joint}"
+      parent="${prefix}${hand_name}"
+      link_name="${prefix}${ee_name}"
+      joint_origin_xyz="${ee_origin_xyz}"
+      joint_origin_rpy="${ee_origin_rpy}"
+      gazebo_preserve_fixed_joint="${gazebo_preserve_fixed_joint}"
     />
   </xacro:macro>

File: src/panda_description/urdf/panda_inertial.xacro (robot description, xacro)
@@ -5,18 +5,18 @@
   <!-- Properties -->
   <!--            -->
-  <xacro:property name="link0_mesh" value="link0"/>
-  <xacro:property name="link1_mesh" value="link1"/>
-  <xacro:property name="link2_mesh" value="link2"/>
-  <xacro:property name="link3_mesh" value="link3"/>
-  <xacro:property name="link4_mesh" value="link4"/>
-  <xacro:property name="link5_mesh" value="link5"/>
-  <xacro:property name="link6_mesh" value="link6"/>
-  <xacro:property name="link7_mesh" value="link7"/>
-  <xacro:property name="hand_mesh" value="hand"/>
-  <xacro:property name="finger_mesh" value="finger"/>
+  <xacro:property name="link0_mesh" value="link0" />
+  <xacro:property name="link1_mesh" value="link1" />
+  <xacro:property name="link2_mesh" value="link2" />
+  <xacro:property name="link3_mesh" value="link3" />
+  <xacro:property name="link4_mesh" value="link4" />
+  <xacro:property name="link5_mesh" value="link5" />
+  <xacro:property name="link6_mesh" value="link6" />
+  <xacro:property name="link7_mesh" value="link7" />
+  <xacro:property name="hand_mesh" value="hand" />
+  <xacro:property name="finger_mesh" value="finger" />
   <!--       -->
   <!-- Macro -->
   <!--       -->
-  <xacro:property name="mesh_offset_rpy" value="0 0 0"/>
+  <xacro:property name="mesh_offset_rpy" value="0 0 0" />
   <xacro:macro name="panda_inertial" params="
     mesh
@@ -25,70 +25,80 @@
     <xacro:if value="${mesh == link0_mesh}">
       <inertial>
-        <origin xyz="-0.025566 -2.87883e-05 0.057332" rpy="${mesh_offset_rpy}"/>
-        <mass value="2.814271300104062"/>
-        <inertia ixx="0.0075390636364814695" iyy="0.010508017427382959" izz="0.009864933638708275" ixy="-1.5053124574783335e-05" ixz="-0.0012144328835738973" iyz="1.0434803501032979e-05"/>
+        <origin xyz="-0.025566 -2.87883e-05 0.057332" rpy="${mesh_offset_rpy}" />
+        <mass value="2.814271300104062" />
+        <inertia ixx="0.0075390636364814695" iyy="0.010508017427382959" izz="0.009864933638708275"
+          ixy="-1.5053124574783335e-05" ixz="-0.0012144328835738973" iyz="1.0434803501032979e-05" />
       </inertial>
     </xacro:if>
     <xacro:if value="${mesh == link1_mesh}">
       <inertial>
-        <origin xyz="-3.72212e-09 -0.0324958 -0.0675818" rpy="${mesh_offset_rpy}"/>
-        <mass value="2.6433170427227215"/>
-        <inertia ixx="0.017405076982879724" iyy="0.015352077935781732" izz="0.005987891663073857" ixy="-8.687986369621078e-09" ixz="-1.6277819062920423e-08" iyz="0.004510855959102245"/>
+        <origin xyz="-3.72212e-09 -0.0324958 -0.0675818" rpy="${mesh_offset_rpy}" />
+        <mass value="2.6433170427227215" />
+        <inertia ixx="0.017405076982879724" iyy="0.015352077935781732" izz="0.005987891663073857"
+          ixy="-8.687986369621078e-09" ixz="-1.6277819062920423e-08" iyz="0.004510855959102245" />
       </inertial>
     </xacro:if>
     <xacro:if value="${mesh == link2_mesh}">
       <inertial>
-        <origin xyz="3.17833e-07 -0.06861 0.0322285" rpy="${mesh_offset_rpy}"/>
-        <mass value="2.6652755331661186"/>
-        <inertia ixx="0.01778694005635383" iyy="0.006044133867952844" izz="0.01571095500455695" ixy="8.70635625879119e-08" ixz="3.752072058394008e-08" iyz="-0.004599490295490376"/>
+        <origin xyz="3.17833e-07 -0.06861 0.0322285" rpy="${mesh_offset_rpy}" />
+        <mass value="2.6652755331661186" />
+        <inertia ixx="0.01778694005635383" iyy="0.006044133867952844" izz="0.01571095500455695"
+          ixy="8.70635625879119e-08" ixz="3.752072058394008e-08" iyz="-0.004599490295490376" />
       </inertial>
     </xacro:if>
     <xacro:if value="${mesh == link3_mesh}">
       <inertial>
-        <origin xyz="0.0469893 0.0316374 -0.031704" rpy="${mesh_offset_rpy}"/>
-        <mass value="2.3293714829045733"/>
-        <inertia ixx="0.0075496764161139766" iyy="0.009680676080191398" izz="0.007944557422008086" ixy="-0.0024320464513492225" ixz="-0.003250815048103007" iyz="-0.0021316282421730694"/>
+        <origin xyz="0.0469893 0.0316374 -0.031704" rpy="${mesh_offset_rpy}" />
+        <mass value="2.3293714829045733" />
+        <inertia ixx="0.0075496764161139766" iyy="0.009680676080191398" izz="0.007944557422008086"
+          ixy="-0.0024320464513492225" ixz="-0.003250815048103007" iyz="-0.0021316282421730694" />
       </inertial>
     </xacro:if>
     <xacro:if value="${mesh == link4_mesh}">
       <inertial>
-        <origin xyz="-0.0360505 0.0337069 0.0319019" rpy="${mesh_offset_rpy}"/>
-        <mass value="2.3104763646281508"/>
-        <inertia ixx="0.007764568814864828" iyy="0.008015776929980149" izz="0.009955882308071066" ixy="0.003371475204045935" ixz="-0.002343621113168248" iyz="0.0022917526161470624"/>
+        <origin xyz="-0.0360505 0.0337069 0.0319019" rpy="${mesh_offset_rpy}" />
+        <mass value="2.3104763646281508" />
+        <inertia ixx="0.007764568814864828" iyy="0.008015776929980149" izz="0.009955882308071066"
+          ixy="0.003371475204045935" ixz="-0.002343621113168248" iyz="0.0022917526161470624" />
       </inertial>
     </xacro:if>
     <xacro:if value="${mesh == link5_mesh}">
       <inertial>
-        <origin xyz="-6.12525e-06 0.0610427 -0.104176" rpy="${mesh_offset_rpy}"/>
-        <mass value="2.6226426154892004"/>
-        <inertia ixx="0.029070538014399377" iyy="0.027638529986528795" izz="0.004251111234400737" ixy="6.208738268725568e-07" ixz="-1.0059151925023392e-05" iyz="-0.007424306477850814"/>
+        <origin xyz="-6.12525e-06 0.0610427 -0.104176" rpy="${mesh_offset_rpy}" />
+        <mass value="2.6226426154892004" />
+        <inertia ixx="0.029070538014399377" iyy="0.027638529986528795" izz="0.004251111234400737"
+          ixy="6.208738268725568e-07" ixz="-1.0059151925023392e-05" iyz="-0.007424306477850814" />
       </inertial>
     </xacro:if>
     <xacro:if value="${mesh == link6_mesh}">
       <inertial>
-        <origin xyz="0.051051 0.00910797 0.0106343" rpy="${mesh_offset_rpy}"/>
-        <mass value="1.5025804886626795"/>
-        <inertia ixx="0.002940555801469018" iyy="0.00392105201248677" izz="0.0054115603870960195" ixy="-0.00042391108351381507" ixz="0.000610007735338717" iyz="0.00012647545430836214"/>
+        <origin xyz="0.051051 0.00910797 0.0106343" rpy="${mesh_offset_rpy}" />
+        <mass value="1.5025804886626795" />
+        <inertia ixx="0.002940555801469018" iyy="0.00392105201248677" izz="0.0054115603870960195"
+          ixy="-0.00042391108351381507" ixz="0.000610007735338717" iyz="0.00012647545430836214" />
       </inertial>
     </xacro:if>
     <xacro:if value="${mesh == link7_mesh}">
       <inertial>
-        <origin xyz="0.0109695 0.0107965 0.0650412" rpy="${mesh_offset_rpy}"/>
-        <mass value="0.5237668134788256"/>
-        <inertia ixx="0.0008621467959726535" iyy="0.0008613100184801048" izz="0.0006961139396618219" ixy="-0.00011871071570425467" ixz="3.866602604509339e-05" iyz="-9.057841649422724e-05"/>
+        <origin xyz="0.0109695 0.0107965 0.0650412" rpy="${mesh_offset_rpy}" />
+        <mass value="0.5237668134788256" />
+        <inertia ixx="0.0008621467959726535" iyy="0.0008613100184801048" izz="0.0006961139396618219"
+          ixy="-0.00011871071570425467" ixz="3.866602604509339e-05" iyz="-9.057841649422724e-05" />
       </inertial>
     </xacro:if>
     <xacro:if value="${mesh == hand_mesh}">
       <inertial>
-        <origin xyz="-6.7624e-06 0.00152435 0.0275912" rpy="${mesh_offset_rpy}"/>
-        <mass value="0.14060765127978503"/>
-        <inertia ixx="0.0005365450414352072" iyy="7.70511954783727e-05" izz="0.0004938176882694914" ixy="1.7911952957732454e-08" ixz="-2.320071910601251e-08" iyz="4.681149945315967e-08"/>
+        <origin xyz="-6.7624e-06 0.00152435 0.0275912" rpy="${mesh_offset_rpy}" />
+        <mass value="0.14060765127978503" />
+        <inertia ixx="0.0005365450414352072" iyy="7.70511954783727e-05" izz="0.0004938176882694914"
+          ixy="1.7911952957732454e-08" ixz="-2.320071910601251e-08" iyz="4.681149945315967e-08" />
       </inertial>
     </xacro:if>
     <xacro:if value="${mesh == finger_mesh}">
       <inertial>
-        <origin xyz="-6.2561e-06 0.00227781 -0.0277116" rpy="${mesh_offset_rpy}"/>
-        <mass value="0.2238453537819424"/>
-        <inertia ixx="6.74804167363695e-05" iyy="6.627189221641395e-05" izz="1.550396267804825e-05" ixy="-4.1027443646025676e-09" ixz="1.8693673970152995e-08" iyz="1.1967548474390802e-05"/>
+        <origin xyz="-6.2561e-06 0.00227781 -0.0277116" rpy="${mesh_offset_rpy}" />
+        <mass value="0.2238453537819424" />
+        <inertia ixx="6.74804167363695e-05" iyy="6.627189221641395e-05" izz="1.550396267804825e-05"
+          ixy="-4.1027443646025676e-09" ixz="1.8693673970152995e-08" iyz="1.1967548474390802e-05" />
       </inertial>
     </xacro:if>
